File: board/board.kicad_pcb (KiCad board)
At the start: 2 copper layers, 21 x 13 mm, 1 part

Commit message: imported legacy version
Parts:
- removed LOGO1: Logo_Open_Hardware_Small, Symbol:OSHW-Symbol_6.7x6mm_SilkScreen
- added C1: 22pF, Capacitor_SMD:C_0603_1608Metric, F.Cu at (86.0, 81.2)
- added C2: 22pF, Capacitor_SMD:C_0603_1608Metric, F.Cu at (85.2, 83.6)
- added C3: 1uF, Capacitor_SMD:C_0603_1608Metric, F.Cu at (91.5, 80.8)
- added C4: 100nF, Capacitor_SMD:C_0603_1608Metric, F.Cu at (84.8, 77.4)
- added J1: 002_SPI, on_edge:on_edge_2x05_device, F.Cu at (77.0, 80.5)
- added J2: 012_CAN, on_edge:on_edge_2x05_host, F.Cu at (98.0, 80.5)
- added U1: MCP2515-xSO, Package_SO:SOIC-18W_7.5x11.6mm_P1.27mm, B.Cu at (87.5, 80.4)
- added Y1: 20MhZ, Crystal:Crystal_SMD_Abracon_ABM8G-4Pin_3.2x2.5mm, F.Cu at (88.2, 83.7)
Routing:
- net GND: track 0.00 -> 37.9 mm, vias 0 -> 1
- net +3V3: track 0.00 -> 35.4 mm, vias 0 -> 4
- net +5V: track 0.00 -> 17.8 mm
- net /controller/INT0: track 0.00 -> 13.7 mm
- net /controller/RESET: track 0.00 -> 12.1 mm, vias 0 -> 2
- net /controller/CAN_RX: track 0.00 -> 7.29 mm, vias 0 -> 1
- net Net-(C2-Pad1): track 0.00 -> 7.27 mm, vias 0 -> 1
- net /controller/INT: track 0.00 -> 7.15 mm, vias 0 -> 1
- net /controller/CAN_TX: track 0.00 -> 6.33 mm, vias 0 -> 1
- net Net-(C1-Pad1): track 0.00 -> 6.09 mm, vias 0 -> 1
- net /controller/MOSI: track 0.00 -> 5.43 mm, vias 0 -> 1
- net /controller/CS: track 0.00 -> 3.99 mm
- net /controller/CLK: track 0.00 -> 3.92 mm, vias 0 -> 1
- net /controller/MISO: track 0.00 -> 2.79 mm, vias 0 -> 1
Other:
- outline, holes or cut-outs redrawn
- rule pad_to_mask_clearance: 0 -> 0.04
- board text added: "osf.002.v0.2"
- board text added: "osf.b087.v0.1"
